Commit message: rviz ros2

File: robot_odometry/urdf/differential_robot.urdf.xacro (robot description, xacro)
@@ -1,4 +1,4 @@
 <?xml version="1.0"?>
-<robot name="differential_robot" xmlns:xacro="http://www.ros.org/wiki/xacro">
+<robot name="real_differential_robot" xmlns:xacro="http://www.ros.org/wiki/xacro">
   <!-- 색상 정의 -->
   <material name="blue"><color rgba="0.0 0.0 0.8 1.0"/></material>
@@ -7,36 +7,62 @@
   <material name="green"><color rgba="0.0 0.8 0.0 1.0"/></material>
   <material name="red"><color rgba="0.8 0.0 0.0 1.0"/></material>
-  <!-- Base -->
+  <material name="gray"><color rgba="0.5 0.5 0.5 1.0"/></material>
+  <!-- 실제 로봇 파라미터 (정확한 측정값) -->
+  <xacro:property name="wheel_radius" value="0.103" />        <!-- 지름 20.6cm = 반지름 10.3cm -->
+  <xacro:property name="wheel_width" value="0.08" />          <!-- 추정값 -->
+  <xacro:property name="wheel_base" value="0.503" />          <!-- 바퀴 간 거리 50.3cm -->
+  <xacro:property name="base_width" value="0.45" />           <!-- 베이스 폭 -->
+  <xacro:property name="base_length" value="0.60" />          <!-- 전후 길이 -->
+  <xacro:property name="base_height" value="0.27" />          <!-- 플랫폼 두께 (두배로) -->
+  <xacro:property name="wheel_forward_offset" value="0.30" /> <!-- 바퀴를 앞쪽에 배치 (전륜구동) -->
+  <xacro:property name="base_ground_clearance" value="0.103" /> <!-- 지상고 -->
+  <!-- Base Link (메인 플랫폼) -->
   <link name="base_link">
     <visual>
-      <origin xyz="0 0 0.05" rpy="0 0 0"/>
-      <geometry><box size="0.3 0.25 0.1"/></geometry>
-      <material name="blue"/>
-    </visual>
-    <collision>
-      <origin xyz="0 0 0.05" rpy="0 0 0"/>
-      <geometry><box size="0.3 0.25 0.1"/></geometry>
-    </collision>
-    <inertial>
-      <mass value="5.0"/>
-      <origin xyz="0 0 0.05"/>
-      <inertia ixx="0.083" ixy="0.0" ixz="0.0" iyy="0.083" iyz="0.0" izz="0.083"/>
-    </inertial>
-  </link>
-  <!-- 왼쪽 바퀴 (전방 좌측) -->
+      <origin xyz="0 0 ${base_ground_clearance + base_height/2}" rpy="0 0 0"/>
+      <geometry>
+        <box size="${base_length} ${base_width} ${base_height}"/>
+      </geometry>
+      <material name="gray"/>
+    </visual>
+    <collision>
+      <origin xyz="0 0 ${base_ground_clearance + base_height/2}" rpy="0 0 0"/>
+      <geometry>
+        <box size="${base_length} ${base_width} ${base_height}"/>
+      </geometry>
+    </collision>
+    <inertial>
+      <mass value="15.0"/>  <!-- 실제 로봇은 더 무거움 -->
+      <origin xyz="0 0 ${base_ground_clearance + base_height/2}"/>
+      <inertia ixx="0.5" ixy="0.0" ixz="0.0" iyy="0.5" iyz="0.0" izz="0.8"/>
+    </inertial>
+  </link>
+  <!-- 왼쪽 바퀴 (에어리스 타이어) -->
   <link name="left_wheel_link">
     <visual>
       <origin xyz="0 0 0" rpy="1.5708 0 0"/>
-      <geometry><cylinder radius="0.065" length="0.04"/></geometry>
+      <geometry>
+        <cylinder radius="${wheel_radius}" length="${wheel_width}"/>
+      </geometry>
       <material name="black"/>
     </visual>
-    <collision>
-      <origin xyz="0 0 0" rpy="1.5708 0 0"/>
-      <geometry><cylinder radius="0.065" length="0.04"/></geometry>
-    </collision>
-    <inertial>
-      <mass value="0.5"/>
-      <origin xyz="0 0 0"/>
-      <inertia ixx="0.001" ixy="0.0" ixz="0.0" iyy="0.001" iyz="0.0" izz="0.001"/>
+    <!-- 에어리스 타이어의 내부 구조 시각화 -->
+    <visual>
+      <origin xyz="0 0 0" rpy="1.5708 0 0"/>
+      <geometry>
+        <cylinder radius="${wheel_radius * 0.6}" length="${wheel_width + 0.01}"/>
+      </geometry>
+      <material name="gray"/>
+    </visual>
+    <collision>
+      <origin xyz="0 0 0" rpy="1.5708 0 0"/>
+      <geometry>
+        <cylinder radius="${wheel_radius}" length="${wheel_width}"/>
+      </geometry>
+    </collision>
+    <inertial>
+      <mass value="2.0"/>  <!-- 큰 바퀴는 더 무거움 -->
+      <origin xyz="0 0 0"/>
+      <inertia ixx="0.02" ixy="0.0" ixz="0.0" iyy="0.02" iyz="0.0" izz="0.02"/>
     </inertial>
   </link>
@@ -44,22 +70,36 @@
     <parent link="base_link"/>
     <child link="left_wheel_link"/>
-    <origin xyz="0.1 0.13 0.0" rpy="0 0 0"/>
+    <!-- 전륜구동: 바퀴를 앞쪽에 배치 -->
+    <origin xyz="${wheel_forward_offset} ${wheel_base/2} ${wheel_radius}" rpy="0 0 0"/>
     <axis xyz="0 1 0"/>
-  </joint>
-  <!-- 오른쪽 바퀴 (전방 우측) -->
+    <dynamics damping="0.1" friction="0.1"/>
+  </joint>
+  <!-- 오른쪽 바퀴 (에어리스 타이어) -->
   <link name="right_wheel_link">
     <visual>
       <origin xyz="0 0 0" rpy="1.5708 0 0"/>
-      <geometry><cylinder radius="0.065" length="0.04"/></geometry>
+      <geometry>
+        <cylinder radius="${wheel_radius}" length="${wheel_width}"/>
+      </geometry>
       <material name="black"/>
     </visual>
-    <collision>
-      <origin xyz="0 0 0" rpy="1.5708 0 0"/>
-      <geometry><cylinder radius="0.065" length="0.04"/></geometry>
-    </collision>
-    <inertial>
-      <mass value="0.5"/>
-      <origin xyz="0 0 0"/>
-      <inertia ixx="0.001" ixy="0.0" ixz="0.0" iyy="0.001" iyz="0.0" izz="0.001"/>
+    <!-- 에어리스 타이어의 내부 구조 시각화 -->
+    <visual>
+      <origin xyz="0 0 0" rpy="1.5708 0 0"/>
+      <geometry>
+        <cylinder radius="${wheel_radius * 0.6}" length="${wheel_width + 0.01}"/>
+      </geometry>
+      <material name="gray"/>
+    </visual>
+    <collision>
+      <origin xyz="0 0 0" rpy="1.5708 0 0"/>
+      <geometry>
+        <cylinder radius="${wheel_radius}" length="${wheel_width}"/>
+      </geometry>
+    </collision>
+    <inertial>
+      <mass value="2.0"/>
+      <origin xyz="0 0 0"/>
+      <inertia ixx="0.02" ixy="0.0" ixz="0.0" iyy="0.02" iyz="0.0" izz="0.02"/>
     </inertial>
   </link>
@@ -67,84 +107,184 @@
     <parent link="base_link"/>
     <child link="right_wheel_link"/>
-    <origin xyz="0.1 -0.13 -0.01" rpy="0 0 0"/>
+    <!-- 전륜구동: 바퀴를 앞쪽에 배치 -->
+    <origin xyz="${wheel_forward_offset} ${-wheel_base/2} ${wheel_radius}" rpy="0 0 0"/>
     <axis xyz="0 1 0"/>
-  </joint>
-<!-- ========== 왼쪽 캐스터 지지대 ========== -->
-<link name="rear_left_caster_holder_link">
-  <visual>
-    <origin xyz="0 0 0" rpy="0 0 0"/>
-    <geometry><box size="0.04 0.04 0.01"/></geometry>
-    <material name="white"/>
-  </visual>
-</link>
-<joint name="rear_left_caster_holder_joint" type="fixed">
-  <parent link="base_link"/>
-  <child link="rear_left_caster_holder_link"/>
-  <origin xyz="-0.13 0.10 -0.005" rpy="0 0 0"/> <!-- 후방 왼쪽 아래 -->
-</joint>
-<!-- ========== 왼쪽 캐스터 바퀴 ========== -->
+    <dynamics damping="0.1" friction="0.1"/>
+  </joint>
 <link name="rear_left_caster_link">
-  <visual>
-    <origin xyz="0 0 -0.025" rpy="0 0 0"/>
-    <geometry><sphere radius="0.02"/></geometry>
-    <material name="white"/>
-  </visual>
-</link>
-<joint name="rear_left_caster_joint" type="fixed">
-  <parent link="rear_left_caster_holder_link"/>
-  <child link="rear_left_caster_link"/>
-  <origin xyz="0 0 0" rpy="0 0 0"/>
-</joint>
-<!-- ========== 오른쪽 캐스터 지지대 ========== -->
-<link name="rear_right_caster_holder_link">
-  <visual>
-    <origin xyz="0 0 0" rpy="0 0 0"/>
-    <geometry><box size="0.04 0.04 0.01"/></geometry>
-    <material name="white"/>
-  </visual>
-</link>
-<joint name="rear_right_caster_holder_joint" type="fixed">
-  <parent link="base_link"/>
-  <child link="rear_right_caster_holder_link"/>
-  <origin xyz="-0.13 -0.10 -0.005" rpy="0 0 0"/> <!-- ← 왼쪽과 z 높이 맞춤 -->
-</joint>
-<!-- ========== 오른쪽 캐스터 바퀴 ========== -->
-<link name="rear_right_caster_link">
-  <visual>
-    <origin xyz="0 0 -0.025" rpy="0 0 0"/>
-    <geometry><sphere radius="0.02"/></geometry>
-    <material name="white"/>
-  </visual>
-</link>
-<joint name="rear_right_caster_joint" type="fixed">
-  <parent link="rear_right_caster_holder_link"/>
-  <child link="rear_right_caster_link"/>
-  <origin xyz="0 0 0" rpy="0 0 0"/>
-</joint>
-  <!-- IMU -->
+    <visual>
+      <origin xyz="0 0 0" rpy="0 0 0"/>
+      <geometry>
+        <sphere radius="0.05"/> </geometry>
+      <material name="white"/>
+    </visual>
+    <visual>
+      <origin xyz="0 0 0.06" rpy="0 0 0"/>
+      <geometry>
+        <box size="0.05 0.08 0.02"/>
+      </geometry>
+      <material name="gray"/>
+    </visual>
+    <collision>
+      <origin xyz="0 0 0" rpy="0 0 0"/>
+      <geometry>
+        <sphere radius="0.05"/>
+      </geometry>
+    </collision>
+    <inertial>
+      <mass value="0.3"/>
+      <origin xyz="0 0 0"/>
+      <inertia ixx="0.001" ixy="0.0" ixz="0.0" iyy="0.001" iyz="0.0" izz="0.001"/>
+    </inertial>
+  </link>
+  <joint name="rear_left_caster_joint" type="fixed">
+    <parent link="base_link"/>
+    <child link="rear_left_caster_link"/>
+    <origin xyz="-0.25 0.2 0.045" rpy="0 0 0"/>
+  </joint>
+  <link name="rear_right_caster_link">
+    <visual>
+      <origin xyz="0 0 0" rpy="0 0 0"/>
+      <geometry>
+        <sphere radius="0.05"/>
+      </geometry>
+      <material name="white"/>
+    </visual>
+    <visual>
+      <origin xyz="0 0 0.06" rpy="0 0 0"/>
+      <geometry>
+        <box size="0.05 0.08 0.02"/>
+      </geometry>
+      <material name="gray"/>
+    </visual>
+    <collision>
+      <origin xyz="0 0 0" rpy="0 0 0"/>
+      <geometry>
+        <sphere radius="0.05"/>
+      </geometry>
+    </collision>
+    <inertial>
+      <mass value="0.3"/>
+      <origin xyz="0 0 0"/>
+      <inertia ixx="0.001" ixy="0.0" ixz="0.0" iyy="0.001" iyz="0.0" izz="0.001"/>
+    </inertial>
+  </link>
+  <joint name="rear_right_caster_joint" type="fixed">
+    <parent link="base_link"/>
+    <child link="rear_right_caster_link"/>
+    <origin xyz="-0.25 -0.2 0.045" rpy="0 0 0"/>
+  </joint>
+  <!-- IMU (베이스 상단 중앙) -->
   <link name="imu_link">
     <visual>
       <origin xyz="0 0 0" rpy="0 0 0"/>
-      <geometry><box size="0.03 0.03 0.01"/></geometry>
+      <geometry>
+        <box size="0.03 0.03 0.01"/>
+      </geometry>
       <material name="green"/>
     </visual>
+    <collision>
+      <origin xyz="0 0 0" rpy="0 0 0"/>
+      <geometry>
+        <box size="0.03 0.03 0.01"/>
+      </geometry>
+    </collision>
+    <inertial>
+      <mass value="0.1"/>
+      <origin xyz="0 0 0"/>
+      <inertia ixx="0.001" ixy="0.0" ixz="0.0" iyy="0.001" iyz="0.0" izz="0.001"/>
+    </inertial>
   </link>
   <joint name="imu_joint" type="fixed">
     <parent link="base_link"/>
     <child link="imu_link"/>
-    <origin xyz="0.0 0.0 0.08" rpy="0 0 0"/>
-  </joint>
-  <!-- 카메라 -->
+    <origin xyz="0.0 0.0 ${base_ground_clearance + base_height + 0.005}" rpy="0 0 0"/>
+  </joint>
+  <!-- 카메라 (전방 상단, 기존 URDF 스타일) -->
   <link name="camera_link">
     <visual>
       <origin xyz="0 0 0" rpy="0 0 0"/>
-      <geometry><box size="0.025 0.09 0.025"/></geometry>
+      <geometry>
+        <box size="0.025 0.09 0.025"/>
+      </geometry>
       <material name="black"/>
     </visual>
+    <collision>
+      <origin xyz="0 0 0" rpy="0 0 0"/>
+      <geometry>
+        <box size="0.025 0.09 0.025"/>
+      </geometry>
+    </collision>
+    <inertial>
+      <mass value="0.1"/>
+      <origin xyz="0 0 0"/>
+      <inertia ixx="0.001" ixy="0.0" ixz="0.0" iyy="0.001" iyz="0.0" izz="0.001"/>
+    </inertial>
   </link>
   <joint name="camera_joint" type="fixed">
     <parent link="base_link"/>
     <child link="camera_link"/>
-    <origin xyz="0.15 0.0 0.113" rpy="0 0.25 0"/> <!-- 전방 상단, 살짝 아래로 기울임 -->
-  </joint>
+    <!-- 전방 끝에 카메라 배치 (전륜구동 바퀴보다 더 앞쪽) -->
+    <origin xyz="${wheel_forward_offset} 0.0 ${base_ground_clearance + base_height + 0.0125}" rpy="0 0.25 0"/>
+  </joint>
+  <!-- Gazebo 플러그인 설정 -->
+  <gazebo reference="base_link">
+    <material>Gazebo/Black</material>
+  </gazebo>
+  <gazebo reference="left_wheel_link">
+    <material>Gazebo/Black</material>
+    <mu1>1.5</mu1>  <!-- 에어리스 타이어의 높은 마찰력 -->
+    <mu2>1.5</mu2>
+    <kp>10000000.0</kp>
+    <kd>1000.0</kd>
+    <minDepth>0.005</minDepth>
+    <maxVel>2.0</maxVel>
+  </gazebo>
+  <gazebo reference="right_wheel_link">
+    <material>Gazebo/Black</material>
+    <mu1>1.5</mu1>
+    <mu2>1.5</mu2>
+    <kp>10000000.0</kp>
+    <kd>1000.0</kd>
+    <minDepth>0.005</minDepth>
+    <maxVel>2.0</maxVel>
+  </gazebo>
+  <!-- 차동구동 컨트롤러 플러그인 -->
+  <gazebo>
+    <plugin name="differential_drive_controller" filename="libgazebo_ros_diff_drive.so">
+      <ros>
+        <namespace>/</namespace>
+        <remapping>cmd_vel:=cmd_vel</remapping>
+        <remapping>odom:=odom</remapping>
+      </ros>
+      <update_rate>50</update_rate>
+      <left_joint>left_wheel_joint</left_joint>
+      <right_joint>right_wheel_joint</right_joint>
+      <wheel_separation>${wheel_base}</wheel_separation>
+      <wheel_diameter>${2*wheel_radius}</wheel_diameter>
+      <max_wheel_torque>30</max_wheel_torque>
+      <max_wheel_acceleration>2.0</max_wheel_acceleration>
+      <command_topic>cmd_vel</command_topic>
+      <publish_odom>true</publish_odom>
+      <publish_odom_tf>true</publish_odom_tf>
+      <publish_wheel_tf>false</publish_wheel_tf>
+      <odometry_frame>odom</odometry_frame>
+      <robot_base_frame>base_link</robot_base_frame>
+    </plugin>
+  </gazebo>
+  <!-- IMU 센서 플러그인 -->
+  <gazebo reference="imu_link">
+    <sensor name="imu_sensor" type="imu">
+      <plugin filename="libgazebo_ros_imu_sensor.so" name="imu_plugin">
+        <ros>
+          <namespace>/</namespace>
+          <remapping>~/out:=imu/data</remapping>
+        </ros>
+        <initial_orientation_as_reference>false</initial_orientation_as_reference>
+      </plugin>
+      <always_on>true</always_on>
+      <update_rate>100</update_rate>
+      <visualize>true</visualize>
+    </sensor>
+  </gazebo>
 </robot>

Commit message: rviz ros2-v2

File: robot_odometry/urdf/differential_robot.urdf.xacro (robot description, xacro)
@@ -1,5 +1,4 @@
 <?xml version="1.0"?>
 <robot name="real_differential_robot" xmlns:xacro="http://www.ros.org/wiki/xacro">
-  <!-- 색상 정의 -->
   <material name="blue"><color rgba="0.0 0.0 0.8 1.0"/></material>
   <material name="black"><color rgba="0.0 0.0 0.0 1.0"/></material>
@@ -8,14 +7,5 @@
   <material name="red"><color rgba="0.8 0.0 0.0 1.0"/></material>
   <material name="gray"><color rgba="0.5 0.5 0.5 1.0"/></material>
-  <!-- 실제 로봇 파라미터 (정확한 측정값) -->
-  <xacro:property name="wheel_radius" value="0.103" />        <!-- 지름 20.6cm = 반지름 10.3cm -->
-  <xacro:property name="wheel_width" value="0.08" />          <!-- 추정값 -->
-  <xacro:property name="wheel_base" value="0.503" />          <!-- 바퀴 간 거리 50.3cm -->
-  <xacro:property name="base_width" value="0.45" />           <!-- 베이스 폭 -->
-  <xacro:property name="base_length" value="0.60" />          <!-- 전후 길이 -->
-  <xacro:property name="base_height" value="0.27" />          <!-- 플랫폼 두께 (두배로) -->
-  <xacro:property name="wheel_forward_offset" value="0.30" /> <!-- 바퀴를 앞쪽에 배치 (전륜구동) -->
-  <xacro:property name="base_ground_clearance" value="0.103" /> <!-- 지상고 -->
-  <!-- Base Link (메인 플랫폼) -->
+  <xacro:property name="wheel_radius" value="0.103" />         <xacro:property name="wheel_width" value="0.08" />             <xacro:property name="wheel_base" value="0.503" />             <xacro:property name="base_width" value="0.45" />             <xacro:property name="base_length" value="0.60" />             <xacro:property name="base_height" value="0.27" />             <xacro:property name="wheel_forward_offset" value="0.30" /> <xacro:property name="base_ground_clearance" value="0.103" /> <xacro:property name="camera_height_offset" value="0.0125" /> <xacro:property name="camera_tilt_angle" value="0.25" />       <link name="world"/>
   <link name="base_link">
     <visual>
@@ -32,11 +22,10 @@
       </geometry>
     </collision>
-    <inertial>
-      <mass value="15.0"/>  <!-- 실제 로봇은 더 무거움 -->
-      <origin xyz="0 0 ${base_ground_clearance + base_height/2}"/>
-      <inertia ixx="0.5" ixy="0.0" ixz="0.0" iyy="0.5" iyz="0.0" izz="0.8"/>
-    </inertial>
   </link>
-  <!-- 왼쪽 바퀴 (에어리스 타이어) -->
+  <joint name="world_to_base_joint" type="fixed">
+    <parent link="world"/>
+    <child link="base_link"/>
+    <origin xyz="0 0 0" rpy="0 0 0"/>
+  </joint>
   <link name="left_wheel_link">
     <visual>
@@ -47,5 +36,4 @@
       <material name="black"/>
     </visual>
-    <!-- 에어리스 타이어의 내부 구조 시각화 -->
     <visual>
       <origin xyz="0 0 0" rpy="1.5708 0 0"/>
@@ -61,19 +49,12 @@
       </geometry>
     </collision>
-    <inertial>
-      <mass value="2.0"/>  <!-- 큰 바퀴는 더 무거움 -->
-      <origin xyz="0 0 0"/>
-      <inertia ixx="0.02" ixy="0.0" ixz="0.0" iyy="0.02" iyz="0.0" izz="0.02"/>
-    </inertial>
   </link>
   <joint name="left_wheel_joint" type="continuous">
     <parent link="base_link"/>
     <child link="left_wheel_link"/>
-    <!-- 전륜구동: 바퀴를 앞쪽에 배치 -->
     <origin xyz="${wheel_forward_offset} ${wheel_base/2} ${wheel_radius}" rpy="0 0 0"/>
     <axis xyz="0 1 0"/>
     <dynamics damping="0.1" friction="0.1"/>
   </joint>
-  <!-- 오른쪽 바퀴 (에어리스 타이어) -->
   <link name="right_wheel_link">
     <visual>
@@ -84,5 +65,4 @@
       <material name="black"/>
     </visual>
-    <!-- 에어리스 타이어의 내부 구조 시각화 -->
     <visual>
       <origin xyz="0 0 0" rpy="1.5708 0 0"/>
@@ -98,23 +78,18 @@
       </geometry>
     </collision>
-    <inertial>
-      <mass value="2.0"/>
-      <origin xyz="0 0 0"/>
-      <inertia ixx="0.02" ixy="0.0" ixz="0.0" iyy="0.02" iyz="0.0" izz="0.02"/>
-    </inertial>
   </link>
   <joint name="right_wheel_joint" type="continuous">
     <parent link="base_link"/>
     <child link="right_wheel_link"/>
-    <!-- 전륜구동: 바퀴를 앞쪽에 배치 -->
     <origin xyz="${wheel_forward_offset} ${-wheel_base/2} ${wheel_radius}" rpy="0 0 0"/>
     <axis xyz="0 1 0"/>
     <dynamics damping="0.1" friction="0.1"/>
   </joint>
-<link name="rear_left_caster_link">
+  <link name="rear_left_caster_link">
     <visual>
       <origin xyz="0 0 0" rpy="0 0 0"/>
       <geometry>
-        <sphere radius="0.05"/> </geometry>
+        <sphere radius="0.05"/>
+      </geometry>
       <material name="white"/>
     </visual>
@@ -132,9 +107,4 @@
       </geometry>
     </collision>
-    <inertial>
-      <mass value="0.3"/>
-      <origin xyz="0 0 0"/>
-      <inertia ixx="0.001" ixy="0.0" ixz="0.0" iyy="0.001" iyz="0.0" izz="0.001"/>
-    </inertial>
   </link>
   <joint name="rear_left_caster_joint" type="fixed">
@@ -164,9 +134,4 @@
       </geometry>
     </collision>
-    <inertial>
-      <mass value="0.3"/>
-      <origin xyz="0 0 0"/>
-      <inertia ixx="0.001" ixy="0.0" ixz="0.0" iyy="0.001" iyz="0.0" izz="0.001"/>
-    </inertial>
   </link>
   <joint name="rear_right_caster_joint" type="fixed">
@@ -175,31 +140,4 @@
     <origin xyz="-0.25 -0.2 0.045" rpy="0 0 0"/>
   </joint>
-  <!-- IMU (베이스 상단 중앙) -->
-  <link name="imu_link">
-    <visual>
-      <origin xyz="0 0 0" rpy="0 0 0"/>
-      <geometry>
-        <box size="0.03 0.03 0.01"/>
-      </geometry>
-      <material name="green"/>
-    </visual>
-    <collision>
-      <origin xyz="0 0 0" rpy="0 0 0"/>
-      <geometry>
-        <box size="0.03 0.03 0.01"/>
-      </geometry>
-    </collision>
-    <inertial>
-      <mass value="0.1"/>
-      <origin xyz="0 0 0"/>
-      <inertia ixx="0.001" ixy="0.0" ixz="0.0" iyy="0.001" iyz="0.0" izz="0.001"/>
-    </inertial>
-  </link>
-  <joint name="imu_joint" type="fixed">
-    <parent link="base_link"/>
-    <child link="imu_link"/>
-    <origin xyz="0.0 0.0 ${base_ground_clearance + base_height + 0.005}" rpy="0 0 0"/>
-  </joint>
-  <!-- 카메라 (전방 상단, 기존 URDF 스타일) -->
   <link name="camera_link">
     <visual>
@@ -216,75 +154,21 @@
       </geometry>
     </collision>
-    <inertial>
-      <mass value="0.1"/>
-      <origin xyz="0 0 0"/>
-      <inertia ixx="0.001" ixy="0.0" ixz="0.0" iyy="0.001" iyz="0.0" izz="0.001"/>
-    </inertial>
   </link>
   <joint name="camera_joint" type="fixed">
     <parent link="base_link"/>
     <child link="camera_link"/>
-    <!-- 전방 끝에 카메라 배치 (전륜구동 바퀴보다 더 앞쪽) -->
-    <origin xyz="${wheel_forward_offset} 0.0 ${base_ground_clearance + base_height + 0.0125}" rpy="0 0.25 0"/>
+    <origin xyz="${wheel_forward_offset} 0.0 ${base_ground_clearance + base_height + camera_height_offset}" rpy="0 ${camera_tilt_angle} 0"/>
   </joint>
-  <!-- Gazebo 플러그인 설정 -->
-  <gazebo reference="base_link">
-    <material>Gazebo/Black</material>
-  </gazebo>
-  <gazebo reference="left_wheel_link">
-    <material>Gazebo/Black</material>
-    <mu1>1.5</mu1>  <!-- 에어리스 타이어의 높은 마찰력 -->
-    <mu2>1.5</mu2>
-    <kp>10000000.0</kp>
-    <kd>1000.0</kd>
-    <minDepth>0.005</minDepth>
-    <maxVel>2.0</maxVel>
-  </gazebo>
-  <gazebo reference="right_wheel_link">
-    <material>Gazebo/Black</material>
-    <mu1>1.5</mu1>
-    <mu2>1.5</mu2>
-    <kp>10000000.0</kp>
-    <kd>1000.0</kd>
-    <minDepth>0.005</minDepth>
-    <maxVel>2.0</maxVel>
-  </gazebo>
-  <!-- 차동구동 컨트롤러 플러그인 -->
-  <gazebo>
-    <plugin name="differential_drive_controller" filename="libgazebo_ros_diff_drive.so">
-      <ros>
-        <namespace>/</namespace>
-        <remapping>cmd_vel:=cmd_vel</remapping>
-        <remapping>odom:=odom</remapping>
-      </ros>
-      <update_rate>50</update_rate>
-      <left_joint>left_wheel_joint</left_joint>
-      <right_joint>right_wheel_joint</right_joint>
-      <wheel_separation>${wheel_base}</wheel_separation>
-      <wheel_diameter>${2*wheel_radius}</wheel_diameter>
-      <max_wheel_torque>30</max_wheel_torque>
-      <max_wheel_acceleration>2.0</max_wheel_acceleration>
-      <command_topic>cmd_vel</command_topic>
-      <publish_odom>true</publish_odom>
-      <publish_odom_tf>true</publish_odom_tf>
-      <publish_wheel_tf>false</publish_wheel_tf>
-      <odometry_frame>odom</odometry_frame>
-      <robot_base_frame>base_link</robot_base_frame>
-    </plugin>
-  </gazebo>
-  <!-- IMU 센서 플러그인 -->
-  <gazebo reference="imu_link">
-    <sensor name="imu_sensor" type="imu">
-      <plugin filename="libgazebo_ros_imu_sensor.so" name="imu_plugin">
-        <ros>
-          <namespace>/</namespace>
-          <remapping>~/out:=imu/data</remapping>
-        </ros>
-        <initial_orientation_as_reference>false</initial_orientation_as_reference>
-      </plugin>
-      <always_on>true</always_on>
-      <update_rate>100</update_rate>
-      <visualize>true</visualize>
-    </sensor>
-  </gazebo>
+  <link name="camera_color_frame"/>
+  <joint name="camera_color_joint" type="fixed">
+    <parent link="camera_link"/>
+    <child link="camera_color_frame"/>
+    <origin xyz="0 0 0" rpy="0 0 0"/>
+  </joint>
+  <link name="camera_color_optical_frame"/>
+  <joint name="camera_color_optical_joint" type="fixed">
+    <parent link="camera_color_frame"/>
+    <child link="camera_color_optical_frame"/>
+    <origin xyz="0 0 0" rpy="-1.5708 0 -1.5708"/>
+     </joint>
 </robot>
